File: muse-dash-pcb/muse-dash-pcb.kicad_pcb (KiCad board)
At the start: 2 copper layers, 84.1 x 47.3 mm, 24 parts, among them SW0 SW_Push, SW1 CherryMX, SW2 CherryMX, SW3 CherryMX, SW4 CherryMX, U1 ATmega32U4-A, Y1 Crystal_GND24

Commit message: general fixes
Routing:
- net SW1: track 50.9 -> 56.1 mm
Changed lines of the file:
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@@
 		(tags "resistor handsolder")
 		(property "Reference" "R3"
-			(at 0 -1.65 0)
+			(at 3.06375 0.22225 0)
 			(layer "F.SilkS")
 			(effects
@@
 		)
 		(property "Value" "R"
-			(at 0 1.65 0)
+			(at 0 2.38125 0)
 			(layer "F.Fab")
 			(effects
@@
 		(tags "capacitor")
 		(property "Reference" "C3"
-			(at 0 -1.68 90)
+			(at 0.2475 3.1535 90)
 			(layer "F.SilkS")
 			(effects
@@
 		(tags "capacitor")
 		(property "Reference" "C1"
-			(at 0 -1.68 360)
+			(at 0.05075 -3.1205 0)
 			(layer "F.SilkS")
 			(effects
@@
 		)
 		(property "Value" "0.1uF"
-			(at 0 1.68 360)
+			(at 0.30475 -1.7235 0)
 			(layer "F.Fab")
 			(effects
@@
 		)
 		(fp_text user "${REFERENCE}"
-			(at 0 0 360)
+			(at 0 0 0)
 			(layer "F.Fab")
 			(effects
@@
 		(tags "fuse handsolder")
 		(property "Reference" "F1"
-			(at 0 -1.82 90)
+			(at -0.0365 3.429 90)
 			(layer "F.SilkS")
 			(effects
@@
 		(tags "capacitor")
 		(property "Reference" "C4"
-			(at 0 -1.68 360)
+			(at 0 2.9935 0)
 			(layer "F.SilkS")
 			(effects
@@
 		)
 		(property "Value" "0.1uF"
-			(at 0 1.68 360)
+			(at 0 1.68 0)
 			(layer "F.Fab")
 			(effects
@@
 		)
 		(fp_text user "${REFERENCE}"
-			(at 0 0 360)
+			(at 0 0 0)
 			(layer "F.Fab")
 			(effects
@@
 		(tags "USB USB_B USB_Mini connector")
 		(property "Reference" "USB1"
-			(at 0 -5 360)
+			(at 0 -5 0)
 			(layer "F.SilkS")
 			(effects
@@
 		)
 		(property "Value" "Molex-0548190589"
-			(at 0 7.5 360)
+			(at -0.767 -6.537 0)
 			(layer "F.Fab")
 			(effects
@@
 		)
 		(fp_text user "${REFERENCE}"
-			(at 0 1.6 360)
+			(at 0 1.6 0)
 			(layer "F.Fab")
 			(effects
@@
 			(at 0 -7.45 0)
 			(layer "F.SilkS")
+			(hide yes)
 			(effects
 				(font
@@
 		)
 		(property "Value" "ATmega32U4-A"
-			(at 0 7.45 0)
+			(at 0.25875 1.2735 0)
 			(layer "F.Fab")
 			(effects
 				(font
-					(size 1 1)
-					(thickness 0.15)
+					(size 0.381 0.381)
+					(thickness 0.0508)
 				)
 			)
@@
 		(tags "resistor handsolder")
 		(property "Reference" "R4"
-			(at 0 -1.65 360)
+			(at -3.06375 -0.1905 0)
 			(layer "F.SilkS")
 			(effects
@@
 		)
 		(property "Value" "10k"
-			(at 0 1.65 360)
+			(at 0 1.65 0)
 			(layer "F.Fab")
 			(effects
@@
 		)
 		(fp_text user "${REFERENCE}"
-			(at 0 0 360)
+			(at 0 0 0)
 			(layer "F.Fab")
 			(effects
@@
 	)
 	(segment
-		(start 158.90875 86.51875)
-		(end 167.8305 77.597)
+		(start 158.877 77.724)
+		(end 159.004 77.597)
 		(width 0.254)
 		(layer "B.Cu")
@@
 	)
 	(segment
-		(start 167.8305 77.597)
-		(end 167.894 77.597)
+		(start 158.877 86.487)
+		(end 158.877 77.724)
 		(width 0.254)
 		(layer "B.Cu")
@@
 	)
 	(segment
-		(start 167.894 77.597)
-		(end 192.913 77.597)
+		(start 158.90875 86.51875)
+		(end 158.877 86.487)
 		(width 0.254)
 		(layer "B.Cu")
@@
 	)
 	(segment
+		(start 159.004 77.597)
+		(end 192.913 77.597)
+		(width 0.254)
+		(layer "B.Cu")
+		(net 18)
+	)
+	(segment
 		(start 198.247 73.394374)
 		(end 198.247 69.469)
@@
 	)
 	(segment
-		(start 203.99375 86.51875)
-		(end 206.121 84.3915)
+		(start 203.99375 79.08925)
+		(end 206.121 76.962)
 		(width 0.254)
 		(layer "B.Cu")
@@
 	)
 	(segment
-		(start 206.121 84.3915)
-		(end 206.121 66.04)
+		(start 206.121 66.04)
+		(end 207.518 64.643)
 		(width 0.254)
 		(layer "B.Cu")
@@
 	)
 	(segment
-		(start 206.121 66.04)
-		(end 207.518 64.643)
+		(start 203.99375 86.51875)
+		(end 203.99375 79.08925)
+		(width 0.254)
+		(layer "B.Cu")
+		(net 20)
+	)
+	(segment
+		(start 206.121 76.962)
+		(end 206.121 66.04)
 		(width 0.254)
 		(layer "B.Cu")
@@
 	)
 	(segment
-		(start 223.8375 86.51875)
-		(end 223.8375 73.7235)
+		(start 223.8375 73.7235)
+		(end 213.868 63.754)
 		(width 0.254)
 		(layer "B.Cu")
@@
 	)
 	(segment
-		(start 223.8375 73.7235)
-		(end 213.868 63.754)
+		(start 223.8375 86.51875)
+		(end 223.8375 73.7235)
 		(width 0.254)
 		(layer "B.Cu")
